File: Heatplate_v1.2/Heatplate_v1.2.kicad_sch (KiCad schematic)
At the start: 42 parts, among them J1 Barrel_Jack_Switch, Q1 WSP4409A, Q2 IRLR8726TRPBF, Q3 SS8050, U1 ATMEGA4809-AFR, U2 AMS1117-5.0

Commit message: BOM
Parts:
- C2, C5: LCSC Part Number C442884 -> C882163
Changed lines of the file:
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@@
       (effects (font (size 1.27 1.27)) hide)
     )
-    (property "LCSC Part Number" "C442884" (at 83.82 41.91 0)
+    (property "LCSC Part Number" "C882163" (at 83.82 41.91 0)
       (effects (font (size 1.27 1.27)) hide)
     )
@@
       (effects (font (size 1.27 1.27)) hide)
     )
-    (property "LCSC Part Number" "C442884" (at 133.35 41.91 0)
-      (effects (font (size 1.27 1.27)) hide)
-    )
+    (property "LCSC Part Number" "C882163" (at 133.35 41.91 0)
+      (effects (font (size 1.27 1.27)) hide)
+    )
